Commit message: update

File: src/simple_object_control/urdf/simple_object.urdf (robot description, URDF)
Before this commit: robot simple_object, 1 links, 0 joints
Links:
- link base_link: geometry visual box size=0.6 0.4 0.3

Commit message: 暂存

File: src/simple_object_control/urdf/simple_object.urdf (robot description, URDF)
Before this commit: robot simple_object, 1 links, 0 joints
Links:
- removed link base_link
- added link body; visual box size=0.6 0.4 0.3
